File: can.kicad_sch (KiCad schematic)
At the start: 11 parts

Commit message: some form of schematic done, still lots to test
Parts:
- gave numbers to parts that had none: 11
Changed lines of the file:
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@@
   (symbol (lib_id "power:GND") (at 171.45 66.675 0) (unit 1)
     (in_bom yes) (on_board yes) (fields_autoplaced)
-    (property "Reference" "#PWR?" (id 0) (at 171.45 73.025 0)
+    (property "Reference" "#PWR0410" (id 0) (at 171.45 73.025 0)
       (effects (font (size 1.27 1.27)) hide)
     )
@@
   (symbol (lib_id "power:GND") (at 119.38 117.475 0) (unit 1)
     (in_bom yes) (on_board yes) (fields_autoplaced)
-    (property "Reference" "#PWR?" (id 0) (at 119.38 123.825 0)
+    (property "Reference" "#PWR0407" (id 0) (at 119.38 123.825 0)
       (effects (font (size 1.27 1.27)) hide)
     )
@@
   (symbol (lib_id "Device:R") (at 119.38 68.58 0) (unit 1)
     (in_bom yes) (on_board yes) (fields_autoplaced)
-    (property "Reference" "R?" (id 0) (at 121.158 67.6715 0)
+    (property "Reference" "R403" (id 0) (at 121.158 67.6715 0)
       (effects (font (size 1.27 1.27)) (justify left))
     )
@@
   (symbol (lib_id "power:+5V") (at 192.405 54.61 0) (unit 1)
     (in_bom yes) (on_board yes) (fields_autoplaced)
-    (property "Reference" "#PWR?" (id 0) (at 192.405 58.42 0)
+    (property "Reference" "#PWR0412" (id 0) (at 192.405 58.42 0)
       (effects (font (size 1.27 1.27)) hide)
     )
@@
   (symbol (lib_id "power:+3.3V") (at 111.125 57.785 0) (unit 1)
     (in_bom yes) (on_board yes) (fields_autoplaced)
-    (property "Reference" "#PWR?" (id 0) (at 111.125 61.595 0)
+    (property "Reference" "#PWR0405" (id 0) (at 111.125 61.595 0)
       (effects (font (size 1.27 1.27)) hide)
     )
@@
   (symbol (lib_id "Device:C") (at 171.45 62.23 0) (unit 1)
     (in_bom yes) (on_board yes) (fields_autoplaced)
-    (property "Reference" "C?" (id 0) (at 174.371 61.3215 0)
+    (property "Reference" "C405" (id 0) (at 174.371 61.3215 0)
       (effects (font (size 1.27 1.27)) (justify left))
     )
@@
   (symbol (lib_id "Device:R") (at 111.125 68.58 0) (unit 1)
     (in_bom yes) (on_board yes) (fields_autoplaced)
-    (property "Reference" "R?" (id 0) (at 112.903 67.6715 0)
+    (property "Reference" "R402" (id 0) (at 112.903 67.6715 0)
       (effects (font (size 1.27 1.27)) (justify left))
     )
@@
   (symbol (lib_id "power:+3.3V") (at 89.535 54.61 0) (unit 1)
     (in_bom yes) (on_board yes) (fields_autoplaced)
-    (property "Reference" "#PWR?" (id 0) (at 89.535 58.42 0)
+    (property "Reference" "#PWR0403" (id 0) (at 89.535 58.42 0)
       (effects (font (size 1.27 1.27)) hide)
     )
@@
   (symbol (lib_id "power:GND") (at 62.865 112.395 0) (unit 1)
     (in_bom yes) (on_board yes) (fields_autoplaced)
-    (property "Reference" "#PWR?" (id 0) (at 62.865 118.745 0)
+    (property "Reference" "#PWR0401" (id 0) (at 62.865 118.745 0)
       (effects (font (size 1.27 1.27)) hide)
     )
@@
   (symbol (lib_id "power:GND") (at 178.435 88.265 0) (unit 1)
     (in_bom yes) (on_board yes) (fields_autoplaced)
-    (property "Reference" "#PWR?" (id 0) (at 178.435 94.615 0)
+    (property "Reference" "#PWR0411" (id 0) (at 178.435 94.615 0)
       (effects (font (size 1.27 1.27)) hide)
     )
@@
   (symbol (lib_id "power:GND") (at 192.405 92.075 0) (unit 1)
     (in_bom yes) (on_board yes) (fields_autoplaced)
-    (property "Reference" "#PWR?" (id 0) (at 192.405 98.425 0)
+    (property "Reference" "#PWR0413" (id 0) (at 192.405 98.425 0)
       (effects (font (size 1.27 1.27)) hide)
     )
@@
   (symbol (lib_id "power:+3.3V") (at 119.38 57.785 0) (unit 1)
     (in_bom yes) (on_board yes) (fields_autoplaced)
-    (property "Reference" "#PWR?" (id 0) (at 119.38 61.595 0)
+    (property "Reference" "#PWR0406" (id 0) (at 119.38 61.595 0)
       (effects (font (size 1.27 1.27)) hide)
     )
@@
   (symbol (lib_id "power:GND") (at 155.575 66.04 0) (unit 1)
     (in_bom yes) (on_board yes) (fields_autoplaced)
-    (property "Reference" "#PWR?" (id 0) (at 155.575 72.39 0)
+    (property "Reference" "#PWR0408" (id 0) (at 155.575 72.39 0)
       (effects (font (size 1.27 1.27)) hide)
     )
@@
   (symbol (lib_id "Device:C") (at 77.47 62.23 0) (unit 1)
     (in_bom yes) (on_board yes) (fields_autoplaced)
-    (property "Reference" "C?" (id 0) (at 80.391 61.3215 0)
+    (property "Reference" "C402" (id 0) (at 80.391 61.3215 0)
       (effects (font (size 1.27 1.27)) (justify left))
     )
@@
   (symbol (lib_id "Device:C") (at 119.38 113.665 0) (unit 1)
     (in_bom yes) (on_board yes) (fields_autoplaced)
-    (property "Reference" "C?" (id 0) (at 122.301 112.7565 0)
+    (property "Reference" "C403" (id 0) (at 122.301 112.7565 0)
       (effects (font (size 1.27 1.27)) (justify left))
     )
@@
   (symbol (lib_id "power:GND") (at 89.535 112.395 0) (unit 1)
     (in_bom yes) (on_board yes) (fields_autoplaced)
-    (property "Reference" "#PWR?" (id 0) (at 89.535 118.745 0)
+    (property "Reference" "#PWR0404" (id 0) (at 89.535 118.745 0)
       (effects (font (size 1.27 1.27)) hide)
     )
@@
   (symbol (lib_id "Interface_CAN_LIN:MCP2562-E-SN") (at 192.405 81.915 0) (unit 1)
     (in_bom yes) (on_board yes) (fields_autoplaced)
-    (property "Reference" "U?" (id 0) (at 194.4244 70.3285 0)
+    (property "Reference" "U402" (id 0) (at 194.4244 70.3285 0)
       (effects (font (size 1.27 1.27)) (justify left))
     )
@@
   (symbol (lib_id "Interface_CAN_LIN:MCP2515-xST") (at 89.535 92.075 0) (unit 1)
     (in_bom yes) (on_board yes) (fields_autoplaced)
-    (property "Reference" "U?" (id 0) (at 91.5544 70.3285 0)
+    (property "Reference" "U401" (id 0) (at 91.5544 70.3285 0)
       (effects (font (size 1.27 1.27)) (justify left))
     )
@@
   (symbol (lib_id "Device:C") (at 180.34 62.23 0) (unit 1)
     (in_bom yes) (on_board yes) (fields_autoplaced)
-    (property "Reference" "C?" (id 0) (at 183.261 61.3215 0)
+    (property "Reference" "C406" (id 0) (at 183.261 61.3215 0)
       (effects (font (size 1.27 1.27)) (justify left))
     )
@@
   (symbol (lib_id "Device:C") (at 68.58 62.23 0) (unit 1)
     (in_bom yes) (on_board yes) (fields_autoplaced)
-    (property "Reference" "C?" (id 0) (at 71.501 61.3215 0)
+    (property "Reference" "C401" (id 0) (at 71.501 61.3215 0)
       (effects (font (size 1.27 1.27)) (justify left))
     )
@@
   (symbol (lib_id "power:+3.3V") (at 166.37 53.975 0) (unit 1)
     (in_bom yes) (on_board yes) (fields_autoplaced)
-    (property "Reference" "#PWR?" (id 0) (at 166.37 57.785 0)
+    (property "Reference" "#PWR0409" (id 0) (at 166.37 57.785 0)
       (effects (font (size 1.27 1.27)) hide)
     )
@@
   (symbol (lib_id "power:GND") (at 68.58 66.675 0) (unit 1)
     (in_bom yes) (on_board yes) (fields_autoplaced)
-    (property "Reference" "#PWR?" (id 0) (at 68.58 73.025 0)
+    (property "Reference" "#PWR0402" (id 0) (at 68.58 73.025 0)
       (effects (font (size 1.27 1.27)) hide)
     )
@@
   (symbol (lib_id "Device:C") (at 155.575 62.23 0) (unit 1)
     (in_bom yes) (on_board yes) (fields_autoplaced)
-    (property "Reference" "C?" (id 0) (at 158.496 61.3215 0)
+    (property "Reference" "C404" (id 0) (at 158.496 61.3215 0)
       (effects (font (size 1.27 1.27)) (justify left))
     )
@@
   (symbol (lib_id "Device:R") (at 62.865 108.585 0) (unit 1)
     (in_bom yes) (on_board yes) (fields_autoplaced)
-    (property "Reference" "R?" (id 0) (at 64.643 107.6765 0)
-      (effects (font (size 1.27 1.27)) (justify left))
-    )
+    (property "Reference" "R401" (id 0) (at 64.643 107.6765 0)
+      (effects (font (size 1.27 1.27)) (justify left))
+    )
