File: cpu.kicad_sch (KiCad schematic)
At the start: 0 parts

Commit message: some form of schematic done, still lots to test
Parts:
- added C601: 1u, Capacitor_SMD:C_0603_1608Metric_Pad1.08x0.95mm_HandSolder, symbol Device:C
- added C602: 100n, Capacitor_SMD:C_0603_1608Metric_Pad1.08x0.95mm_HandSolder, symbol Device:C
- added C603, C604: 10n, Capacitor_SMD:C_0603_1608Metric_Pad1.08x0.95mm_HandSolder, symbol Device:C
- added D601: RSX301L-30TE25, good_things:SOD-106, symbol Device:D
- added Q601, Q602: KST5551, Package_TO_SOT_SMD:SOT-23_Handsoldering, symbol Device:Q_NPN_BEC
- added R601, R602, R603, R604, R605, R606, R607, R608, R609, R610, R611: 470, Resistor_SMD:R_0603_1608Metric_Pad0.98x0.95mm_HandSolder, symbol Device:R_Small
- added R612: 1k, Resistor_SMD:R_0603_1608Metric_Pad0.98x0.95mm_HandSolder, symbol Device:R
- added R613: 10k, Resistor_SMD:R_0603_1608Metric_Pad0.98x0.95mm_HandSolder, symbol Device:R
- added U601, U602: MAN74A, Display_7Segment:MAN71A, symbol Display_Character:MAN74A
- added U603: Pico, MCU_RaspberryPi_and_Boards:RPi_Pico_SMD_TH, symbol MCU_RaspberryPi_and_Boards:Pico
- added U604: LM358, symbol Amplifier_Operational:LM358
Connections:
- new net +3.3VA: C601.1, C602.1, R612.1, U604.8 (V+)
- new net +3V3: U603.36 (3V3)
- new net +5V: D601.2 (A)
- new net 7SEG_A: R603.1, U601.14 (A), U602.14 (A)
- new net 7SEG_A_PRER: R603.2, U603.12 (GPIO9)
- new net 7SEG_B: R604.1, U601.13 (B), U602.13 (B)
- new net 7SEG_B_PRER: R604.2, U603.14 (GPIO10)
- new net 7SEG_C: R605.1, U601.8 (C), U602.8 (C)
- new net 7SEG_C_PRER: R605.2, U603.15 (GPIO11)
- new net 7SEG_D: R606.1, U601.7 (D), U602.7 (D)
- new net 7SEG_DIG0: Q602.3 (C), U602.12 (CC), U602.4 (CC)
- new net 7SEG_DIG0_BASE: Q602.1 (B), R601.1
- new net 7SEG_DIG0_PRER: R601.2, U603.10 (GPIO7)
- new net 7SEG_DIG1: Q601.3 (C), U601.12 (CC), U601.4 (CC)
- new net 7SEG_DIG1_BASE: Q601.1 (B), R602.1
- new net 7SEG_DIG1_PRER: R602.2, U603.11 (GPIO8)
- new net 7SEG_D_PRER: R606.2, U603.16 (GPIO12)
- new net 7SEG_E: R607.1, U601.6 (E), U602.6 (E)
- new net 7SEG_E_PRER: R607.2, U603.17 (GPIO13)
- new net 7SEG_F: R608.1, U601.1 (F), U602.1 (F)
- new net 7SEG_F_PRER: R608.2, U603.19 (GPIO14)
- new net 7SEG_G: R609.1, U601.2 (G), U602.2 (G)
- new net 7SEG_G_PRER: R609.2, U603.20 (GPIO15)
- new net ADC0: R611.2
- new net ADC1: R610.2
- new net ADC_VREF: U603.35 (ADC_VREF), U604.1, U604.2 (-), U604.6 (-), U604.7
- new net ADC_VREF_DIV: R612.2, R613.1, U604.3 (+), U604.5 (+)
- new net CLK_16M_CAN: U603.27 (GPIO21)
- new net GND: Q601.2 (E), Q602.2 (E), U603.13 (GND), U603.18 (GND), U603.23 (GND), U603.28 (GND), U603.3 (GND), U603.38 (GND), U603.42 (GND), U603.8 (GND)
- new net GNDA: C601.2, C602.2, C603.2, C604.2, R613.2, U603.33 (AGND), U604.4 (V-)
- new net MOTOR_CTRL: U603.26 (GPIO20)
- new net PICO_ADC0: C604.1, R611.1, U603.31 (GPIO26_ADC0)
- new net PICO_ADC1: C603.1, R610.1, U603.32 (GPIO27_ADC1)
- new net ROTARY_COFFEE0: U603.22 (GPIO17)
- new net ROTARY_COFFEE1: U603.21 (GPIO16)
- new net ROTARY_WATER0: U603.25 (GPIO19)
- new net ROTARY_WATER1: U603.24 (GPIO18)
- new net SOLENOID_CTRL: U603.29 (GPIO22)
- new net SPI0_PICO_SCLK: U603.4 (GPIO2)
- new net SPI0_PICO_SI: U603.1 (GPIO0)
- new net SPI0_PICO_SO: U603.5 (GPIO3)
- new net VSYS: D601.1 (K), U603.39 (VSYS)
- new net ~{CAN_INT}: U603.6 (GPIO4)
- new net ~{SPI0_PICO_CS}: U603.2 (GPIO1)
- no-connect marks 0 -> 9
Other:
- note added: "CS can prob be moved to another pin, however check this thorougly in SW... CS can be moved freely other pins can also be moved to other spi pins (+4 on gpio)"
- note added: "Select another 7seg. should be common cathode Also make sure to use some kind of right angle footprint"
- note added: "Verify that this generates 3v 2-3mA load (1k ohm)"
- note added: "verify stabillity of amp increase R if unstable"
