File: test_high_gain_amp/test_high_gain_amp.kicad_sch (KiCad schematic)
At the start: 17 parts

Commit message: Finish 60dB amp prototype
Parts:
- removed J?: Conn_01x05, TerminalBlock:TerminalBlock_bornier-5_P5.08mm, symbol Connector_Generic:Conn_01x05
- added J101: Conn_01x06, TerminalBlock:TerminalBlock_bornier-6_P5.08mm, symbol Connector_Generic:Conn_01x06
- added RV101, RV102: 1M, Potentiometer_THT:Potentiometer_ACP_CA6-H2,5_Horizontal, symbol Device:R_Potentiometer
- Q101: renamed from Q?; footprint (none) -> Package_TO_SOT_SMD:SOT-23_Handsoldering
- gave numbers to parts that had none: 15
Connections:
- net 3v3a_regin is gone; now on net +5V: C103.1, FB101.2, U102.3 (IN)
- net +3.3VA: now also J101.4 (Pin_4), RV101.1
- net +5V: no longer FB101.1, Q101.2 (S)
- net GND: now also J101.3 (Pin_3), J101.5 (Pin_5), RV102.2
- net inn: now reaches C105.1, R105.1, U101.4 (-)
- net inn: now also J101.1 (Pin_1)
- net out: now reaches C105.2, J102.1 (In), R105.2, U101.1
- net vin: now reaches Q101.3 (D)
- net vin: now also J101.6 (Pin_6)
- net inp: now reaches C101.2, R101.2, R102.1, R104.2, U101.3 (+)
- net inp: now also J101.2 (Pin_2), RV101.2, RV102.1
- net vprot_gate: now reaches Q101.1 (G), R103.1
- new net vprot: FB101.1, Q101.2 (S)
- no-connect marks 0 -> 2
Other:
- moved on the sheet: R102, R103
